File: Sprite_CC1310_Development.sch (EAGLE design)
At the start: 68 parts, among them U1 NCP1402

Commit message: need new boost converter, obsolete component :(
Parts:
- removed COAX, COAX1: 734120110, con-coax:734120110
- added R18: 10k, SparkFun:RESISTOR0402-RES
- added U$3, U$7: MM5329-2700, MM5329-2700:MM5329-2700
- added U$8: L6920, L6920:L6920
- L1, L3: device SparkFun:INDUCTOR0402 -> SparkFun:INDUCTOR0603
Connections:
- new net N$40: U$8.FB, U$8.OUT
- new net N$41: R18.1, U$8.SHDN
- net GND: now also U$3.GND1, U$3.GND2, U$3.GND3, U$7.GND1, U$7.GND2, U$7.GND3, U$8.GND; no longer COAX.2, COAX1.2
- net N$14: now also U$7.SIG; no longer COAX1.1
- net N$26: now also U$3.SIG; no longer COAX.1
- net SOLAR_CELLS: now also R18.2
Other:
- moved on the sheet: C18, C19, C21, D1, GPS, L3, LED3, R10, R11, R12, R15, R16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

Commit message: updated boost regulator
Parts:
- removed C19: 10 uF, SparkFun:CAP0402-CAP
- removed C21: 68 uF, SparkFun:CAP1206
- removed D1: MBRA140, SparkFun:DIODESOD
- removed L3: 47uH, SparkFun:INDUCTOR0603
- removed U1: NCP1402, SparkFun:V_REG_NCP1400SOT23-5
- added C22, C23: 47 uF, SparkFun:CAP1206
- added L4: 47uH, SparkFun:INDUCTOR0603
Connections:
- removed net N$16: D1.A, L3.2, U1.LX
- removed net N$40: U$8.FB, U$8.OUT
- new net N$48: L4.1, U$8.LX
- net GND: now also C22.2, C23.2; no longer C19.2, C21.2, U1.GND
- net SOLAR_CELLS: now also C22.1, L4.2; no longer C19.1, L3.1
- net VDDS: now also C23.1, U$8.FB, U$8.OUT; no longer C21.1, D1.C, U1.EN, U1.OUT
Other:
- note removed: "consider different boost converter"
- moved on the sheet: C20, FRONT_PANEL, R18, REAR_PANEL

Commit message: BOM
Parts:
- C22, C23: device SparkFun:CAP1206 -> SparkFun:CAP0805
Other:
- moved on the sheet: C20, C22, C23, FRONT_PANEL, L4, R18, REAR_PANEL

Commit message: cleaning up
Parts:
- renumbered SER3635CT-ND to TSX3225
Changed lines of the file:
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@@
 <part name="GND12" library="SparkFun" deviceset="GND" device=""/>
 <part name="GND13" library="SparkFun" deviceset="GND" device=""/>
-<part name="SER3635CT-ND" library="TSX-3225" deviceset="TSX-3225" device=""/>
+<part name="TSX3225" library="TSX-3225" deviceset="TSX-3225" device=""/>
 <part name="GND14" library="SparkFun" deviceset="GND" device=""/>
 <part name="R2" library="SparkFun" deviceset="RESISTOR" device="0402-RES" value="3.3k"/>
@@
 <instance part="GND12" gate="1" x="25.4" y="76.2"/>
 <instance part="GND13" gate="1" x="40.64" y="76.2"/>
-<instance part="SER3635CT-ND" gate="G$1" x="147.32" y="27.94"/>
+<instance part="TSX3225" gate="G$1" x="147.32" y="27.94"/>
 <instance part="GND14" gate="1" x="147.32" y="10.16"/>
 <instance part="R2" gate="G$1" x="60.96" y="78.74" smashed="yes" rot="R180">
@@
 </segment>
 <segment>
-<pinref part="SER3635CT-ND" gate="G$1" pin="2"/>
-<pinref part="SER3635CT-ND" gate="G$1" pin="4"/>
+<pinref part="TSX3225" gate="G$1" pin="2"/>
+<pinref part="TSX3225" gate="G$1" pin="4"/>
 <wire x1="144.78" y1="17.78" x2="147.32" y2="15.24" width="0.1524" layer="91"/>
 <pinref part="GND14" gate="1" pin="GND"/>
@@
 </segment>
 <segment>
-<pinref part="SER3635CT-ND" gate="G$1" pin="3"/>
+<pinref part="TSX3225" gate="G$1" pin="3"/>
 <wire x1="154.94" y1="27.94" x2="162.56" y2="27.94" width="0.1524" layer="91"/>
 <label x="154.94" y="27.94" size="1.778" layer="95"/>
@@
 </segment>
 <segment>
-<pinref part="SER3635CT-ND" gate="G$1" pin="1"/>
+<pinref part="TSX3225" gate="G$1" pin="1"/>
 <wire x1="139.7" y1="27.94" x2="132.08" y2="27.94" width="0.1524" layer="91"/>
 <label x="132.08" y="27.94" size="1.778" layer="95"/>

Commit message: Updated matching network
Parts:
- removed R14, R16: 0, SparkFun:RESISTOR0603-RES
- added C19: 104 pF, SparkFun:CAP0603-CAP
- added L3: 2.2 nH, SparkFun:INDUCTOR0603
- L2: value 5.6 nH -> DNP
- R17: value 0 -> DNP
Connections:
- net ANTENNA: now also C19.2; no longer R14.2
- net GND: now also C19.1, L3.1; no longer R14.1, R16.1
- net N$15: now also L3.2; no longer R16.2
Changed lines of the file:
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@@
 <grid distance="0.1" unitdist="inch" unit="inch" style="lines" multiple="1" display="no" altdistance="0.01" altunitdist="inch" altunit="inch"/>
 <layers>
-<layer number="1" name="Top" color="4" fill="1" visible="yes" active="no"/>
-<layer number="2" name="Route2" color="1" fill="3" visible="yes" active="no"/>
-<layer number="15" name="Route15" color="4" fill="6" visible="yes" active="no"/>
-<layer number="16" name="Bottom" color="1" fill="1" visible="yes" active="no"/>
-<layer number="17" name="Pads" color="2" fill="1" visible="yes" active="no"/>
-<layer number="18" name="Vias" color="2" fill="1" visible="yes" active="no"/>
-<layer number="19" name="Unrouted" color="6" fill="1" visible="yes" active="no"/>
-<layer number="20" name="Dimension" color="24" fill="1" visible="yes" active="no"/>
-<layer number="21" name="tPlace" color="7" fill="1" visible="yes" active="no"/>
-<layer number="22" name="bPlace" color="7" fill="1" visible="yes" active="no"/>
-<layer number="23" name="tOrigins" color="15" fill="1" visible="yes" active="no"/>
-<layer number="24" name="bOrigins" color="15" fill="1" visible="yes" active="no"/>
-<layer number="25" name="tNames" color="7" fill="1" visible="yes" active="no"/>
-<layer number="26" name="bNames" color="7" fill="1" visible="yes" active="no"/>
-<layer number="27" name="tValues" color="7" fill="1" visible="yes" active="no"/>
-<layer number="28" name="bValues" color="7" fill="1" visible="yes" active="no"/>
+<layer number="1" name="Top" color="4" fill="1" visible="no" active="no"/>
+<layer number="2" name="Route2" color="1" fill="3" visible="no" active="no"/>
+<layer number="15" name="Route15" color="4" fill="6" visible="no" active="no"/>
+<layer number="16" name="Bottom" color="1" fill="1" visible="no" active="no"/>
+<layer number="17" name="Pads" color="2" fill="1" visible="no" active="no"/>
+<layer number="18" name="Vias" color="2" fill="1" visible="no" active="no"/>
+<layer number="19" name="Unrouted" color="6" fill="1" visible="no" active="no"/>
+<layer number="20" name="Dimension" color="24" fill="1" visible="no" active="no"/>
+<layer number="21" name="tPlace" color="7" fill="1" visible="no" active="no"/>
+<layer number="22" name="bPlace" color="7" fill="1" visible="no" active="no"/>
+<layer number="23" name="tOrigins" color="15" fill="1" visible="no" active="no"/>
+<layer number="24" name="bOrigins" color="15" fill="1" visible="no" active="no"/>
+<layer number="25" name="tNames" color="7" fill="1" visible="no" active="no"/>
+<layer number="26" name="bNames" color="7" fill="1" visible="no" active="no"/>
+<layer number="27" name="tValues" color="7" fill="1" visible="no" active="no"/>
+<layer number="28" name="bValues" color="7" fill="1" visible="no" active="no"/>
 <layer number="29" name="tStop" color="7" fill="3" visible="no" active="no"/>
 <layer number="30" name="bStop" color="7" fill="6" visible="no" active="no"/>
@@
 <layer number="35" name="tGlue" color="7" fill="4" visible="no" active="no"/>
 <layer number="36" name="bGlue" color="7" fill="5" visible="no" active="no"/>
-<layer number="37" name="tTest" color="7" fill="1" visible="yes" active="no"/>
-<layer number="38" name="bTest" color="7" fill="1" visible="yes" active="no"/>
+<layer number="37" name="tTest" color="7" fill="1" visible="no" active="no"/>
+<layer number="38" name="bTest" color="7" fill="1" visible="no" active="no"/>
 <layer number="39" name="tKeepout" color="4" fill="11" visible="no" active="no"/>
 <layer number="40" name="bKeepout" color="1" fill="11" visible="no" active="no"/>
@@
 <layer number="44" name="Drills" color="7" fill="1" visible="no" active="no"/>
 <layer number="45" name="Holes" color="7" fill="1" visible="no" active="no"/>
-<layer number="46" name="Milling" color="3" fill="1" visible="yes" active="no"/>
-<layer number="47" name="Measures" color="7" fill="1" visible="yes" active="no"/>
-<layer number="48" name="Document" color="7" fill="1" visible="yes" active="no"/>
-<layer number="49" name="Reference" color="7" fill="1" visible="yes" active="no"/>
-<layer number="50" name="dxf" color="7" fill="1" visible="yes" active="no"/>
-<layer number="51" name="tDocu" color="7" fill="1" visible="yes" active="no"/>
-<layer number="52" name="bDocu" color="7" fill="1" visible="yes" active="no"/>
-<layer number="53" name="tGND_GNDA" color="7" fill="9" visible="yes" active="no"/>
-<layer number="54" name="bGND_GNDA" color="1" fill="9" visible="yes" active="no"/>
-<layer number="56" name="wert" color="7" fill="1" visible="yes" active="no"/>
-<layer number="57" name="tCAD" color="7" fill="1" visible="yes" active="no"/>
-<layer number="59" name="tCarbon" color="7" fill="1" visible="yes" active="no"/>
-<layer number="60" name="bCarbon" color="7" fill="1" visible="yes" active="no"/>
+<layer number="46" name="Milling" color="3" fill="1" visible="no" active="no"/>
+<layer number="47" name="Measures" color="7" fill="1" visible="no" active="no"/>
+<layer number="48" name="Document" color="7" fill="1" visible="no" active="no"/>
+<layer number="49" name="Reference" color="7" fill="1" visible="no" active="no"/>
+<layer number="50" name="dxf" color="7" fill="1" visible="no" active="no"/>
+<layer number="51" name="tDocu" color="7" fill="1" visible="no" active="no"/>
+<layer number="52" name="bDocu" color="7" fill="1" visible="no" active="no"/>
+<layer number="53" name="tGND_GNDA" color="7" fill="9" visible="no" active="no"/>
+<layer number="54" name="bGND_GNDA" color="1" fill="9" visible="no" active="no"/>
+<layer number="56" name="wert" color="7" fill="1" visible="no" active="no"/>
+<layer number="57" name="tCAD" color="7" fill="1" visible="no" active="no"/>
+<layer number="59" name="tCarbon" color="7" fill="1" visible="no" active="no"/>
+<layer number="60" name="bCarbon" color="7" fill="1" visible="no" active="no"/>
 <layer number="88" name="SimResults" color="9" fill="1" visible="yes" active="yes"/>
 <layer number="89" name="SimProbes" color="9" fill="1" visible="yes" active="yes"/>
@@
 <part name="R21" library="SparkFun" deviceset="RESISTOR" device="0603-RES" value="0"/>
 <part name="R22" library="SparkFun" deviceset="RESISTOR" device="0603-RES" value="0"/>
-<part name="L2" library="SparkFun" deviceset="INDUCTOR" device="0603" value="5.6 nH"/>
+<part name="L2" library="SparkFun" deviceset="INDUCTOR" device="0603" value="DNP"/>
 <part name="R13" library="SparkFun" deviceset="RESISTOR" device="0603-RES" value="0"/>
-<part name="R14" library="SparkFun" deviceset="RESISTOR" device="0603-RES" value="0"/>
+<part name="C19" library="SparkFun" deviceset="CAP" device="0603-CAP" value="104 pF"/>
 <part name="R15" library="SparkFun" deviceset="RESISTOR" device="0603-RES" value="0"/>
-<part name="R16" library="SparkFun" deviceset="RESISTOR" device="0603-RES" value="0"/>
+<part name="L3" library="SparkFun" deviceset="INDUCTOR" device="0603" value="2.2 nH"/>
 <part name="GND28" library="SparkFun" deviceset="GND" device=""/>
-<part name="R17" library="SparkFun" deviceset="RESISTOR" device="0603-RES" value="0"/>
+<part name="R17" library="SparkFun" deviceset="RESISTOR" device="0603-RES" value="DNP"/>
 <part name="GND29" library="SparkFun" deviceset="GND" device=""/>
 <part name="U$5" library="johanson_gps_chip" deviceset="JOHANSON_GPS_CHIP" device=""/>
@@
 <attribute name="VALUE" x="19.05" y="109.982" size="1.778" layer="96" rot="R180"/>
 </instance>
-<instance part="R14" gate="G$1" x="12.7" y="116.84" smashed="yes" rot="R270">
-<attribute name="NAME" x="14.1986" y="118.11" size="1.778" layer="95" rot="R270"/>
-<attribute name="VALUE" x="9.398" y="118.11" size="1.778" layer="96" rot="R270"/>
+<instance part="C19" gate="G$1" x="12.7" y="116.84" smashed="yes">
+<attribute name="NAME" x="13.97" y="120.8786" size="1.778" layer="95"/>
+<attribute name="VALUE" x="13.97" y="113.538" size="1.778" layer="96"/>
 </instance>
 <instance part="R15" gate="G$1" x="363.22" y="210.82" smashed="yes" rot="R180">
@@
 <attribute name="VALUE" x="367.03" y="214.122" size="1.778" layer="96" rot="R180"/>
 </instance>
-<instance part="R16" gate="G$1" x="373.38" y="220.98" smashed="yes" rot="R270">
-<attribute name="NAME" x="369.7986" y="222.25" size="1.778" layer="95" rot="R270"/>
-<attribute name="VALUE" x="375.158" y="219.71" size="1.778" layer="96" rot="R270"/>
+<instance part="L3" gate="G$1" x="373.38" y="218.44" smashed="yes">
+<attribute name="NAME" x="369.57" y="219.9386" size="1.778" layer="95"/>
+<attribute name="VALUE" x="374.65" y="212.598" size="1.778" layer="96"/>
 </instance>
 <instance part="GND28" gate="1" x="373.38" y="228.6" rot="R180"/>
@@
 <segment>
 <pinref part="GND46" gate="1" pin="GND"/>
-<pinref part="R14" gate="G$1" pin="1"/>
+<pinref part="C19" gate="G$1" pin="1"/>
 <wire x1="12.7" y1="124.46" x2="12.7" y2="121.92" width="0.1524" layer="91"/>
 </segment>
 <segment>
-<pinref part="R16" gate="G$1" pin="1"/>
+<pinref part="L3" gate="G$1" pin="1"/>
 <pinref part="GND28" gate="1" pin="GND"/>
 </segment>
@@
 <pinref part="R15" gate="G$1" pin="1"/>
 <wire x1="368.3" y1="210.82" x2="373.38" y2="210.82" width="0.1524" layer="91"/>
-<pinref part="R16" gate="G$1" pin="2"/>
-<wire x1="373.38" y1="210.82" x2="373.38" y2="215.9" width="0.1524" layer="91"/>
+<pinref part="L3" gate="G$1" pin="2"/>
 <pinref part="U$5" gate="G$1" pin="SIG"/>
 <wire x1="373.38" y1="205.74" x2="373.38" y2="210.82" width="0.1524" layer="91"/>
@@
 <junction x="12.7" y="17.78"/>
 <pinref part="R13" gate="G$1" pin="2"/>
-<pinref part="R14" gate="G$1" pin="2"/>
-<wire x1="12.7" y1="106.68" x2="12.7" y2="111.76" width="0.1524" layer="91"/>
+<pinref part="C19" gate="G$1" pin="2"/>
+<wire x1="12.7" y1="106.68" x2="12.7" y2="114.3" width="0.1524" layer="91"/>
 <wire x1="12.7" y1="63.5" x2="12.7" y2="106.68" width="0.1524" layer="91"/>
 <junction x="12.7" y="63.5"/>
