File: Eagle/Sprite_CC1310_Development.sch (EAGLE design)
At the start: 68 parts

Commit message: Fixed HDMI
Parts:
- removed U$1: HDMID, HDMID:HDMID
- added R14, R16: 0, SparkFun:RESISTOR0603-RES
- added U$9: HDMID, HDMID:HDMID
Connections:
- new net N$16: R16.2, U$7.SIG
- new net N$40: R14.1, U$3.SIG
- net GND: now also U$9.1, U$9.FOOT1, U$9.FOOT2, U$9.FOOT3, U$9.FOOT4; no longer U$1.19, U$1.FOOT1, U$1.FOOT2, U$1.FOOT3, U$1.FOOT4
- net JTAG_TCKC: now also U$9.14, U$9.15; no longer U$1.5, U$1.6
- net JTAG_TMSC: now also U$9.16, U$9.17; no longer U$1.3, U$1.4
- net N$14: now also R16.1; no longer U$7.SIG
- net N$26: now also R14.2; no longer U$3.SIG
- net RESET: now also U$9.6, U$9.7; no longer U$1.13, U$1.14
- net RXD: now also U$9.2, U$9.3; no longer U$1.17, U$1.18
- net SWO: now also U$9.8, U$9.9; no longer U$1.11, U$1.12
- net TDI: now also U$9.10, U$9.11; no longer U$1.10, U$1.9
- net TDO: now also U$9.12, U$9.13; no longer U$1.7, U$1.8
- net TXD: now also U$9.4, U$9.5; no longer U$1.15, U$1.16
- net VDDS: now also U$9.18, U$9.19; no longer U$1.1, U$1.2

Commit message: updated boost converter, eliminated unnecessary tuning components, rotated oscillator, updated solar pads
Parts:
- removed L2: DNP, SparkFun:INDUCTOR0603
- removed R13, R14, R15, R16, R21, R22: 0, SparkFun:RESISTOR0603-RES
- removed R17: DNP, SparkFun:RESISTOR0603-RES
- removed R18: 10k, SparkFun:RESISTOR0402-RES
- removed U$3, U$7: MM5329-2700, MM5329-2700:MM5329-2700
- L4: value 47uH -> 10uH; device SparkFun:INDUCTOR0603 -> ASPI-0315FS:ASPI-0315FS
Connections:
- removed net N$14: R15.2, R16.1, R17.1, R22.1
- removed net N$16: R16.2, U$7.SIG
- removed net N$25: GPS.RFIN, R22.2
- removed net N$26: L2.1, R13.1, R14.2, R21.2
- removed net N$27: C26.1, R21.1
- removed net N$40: R14.1, U$3.SIG
- removed net N$41: R18.1, U$8.SHDN
- net ANTENNA: now also C26.1; no longer R13.2
- net GND: no longer L2.2, R17.2, U$3.GND1, U$3.GND2, U$3.GND3, U$7.GND1, U$7.GND2, U$7.GND3
- net N$15: now also GPS.RFIN; no longer R15.1
- net SOLAR_CELLS: now also U$8.SHDN; no longer R18.2
Other:
- moved on the sheet: C18, C19, GPS, L3, L4, LED3, R10, R11, R12, R9

Commit message: still need to add breakouts
Parts:
- removed LS1: LIGHTSENSORALS, SparkFun-Sensors:LIGHTSENSORALS
- removed U$9: HDMID, HDMID:HDMID
- added C21: 0.1 uF, SparkFun:CAP0402-CAP
- added J2: CORTEX_DEBUG_SMD, SparkFun-Connectors:CORTEX_DEBUG_SMD
- added JP1, JP2: (no value), SparkFun-Connectors:M14
- added NPN: MMDT3904, mmdt3904:MMDT3904
- added PNP: MMDT3906, mmdt3906:MMDT3906
- added R13, R15: 330, SparkFun:RESISTOR0402-RES
- added R14: 10k, SparkFun:RESISTOR0402-RES
- added R16, R21, R22, R23: 0, SparkFun:RESISTOR0603-RES
- added R17, R18, R24, R25: DNP, SparkFun:RESISTOR0603-RES
- added SCHTOKKY: STPS1L30MF, stps1l30mf:STPS1L30MF
- added SI7021: SI7021, si7021:SI7021
- added SUPERCAPACITOR: SUPERCAP1, supercap1:SUPERCAP1
- added U$1, U$3: MM5329-2700, MM5329-2700:MM5329-2700
- FRONT_PANEL, REAR_PANEL: value ALTA_CELL -> SOLARMD; device ALTA_CELL:ALTA_CELL -> solarmd:SOLARMD
- R20: value 331 -> 330
- R7: value 10k -> 330
Connections:
- removed net ADC0: LS1.E1, MICROCONTROLLER.36, R7.1
- new net BPNP: NPN.C2, R14.2, R15.1
- new net IMUGND: C13.2, C14.2, C15.2, C16.2, C17.2, IMU.GND, IMU.RES, NPN.C1, SI7021.GND
- new net N$14: NPN.B2, R7.2
- new net N$16: NPN.B1, R13.1
- new net N$25: PNP.B2, R15.2
- new net N$26: R16.2, R17.1, R18.2, R21.1
- new net N$27: C26.1, R21.2
- new net N$40: R18.1, U$1.SIG
- new net N$41: GPS.RFIN, R22.1
- new net N$49: R22.2, R23.1, R24.1, R25.1
- new net N$50: R25.2, U$3.SIG
- new net SUPERCAP: C22.1, L4.2, MICROCONTROLLER.36, SCHTOKKY.C, SUPERCAPACITOR.+, U$8.SHDN
- new net TRANS: MICROCONTROLLER.31, R13.2, R7.1
- new net VSENSE: GPS.VCC@2, GPS.VCC@58, LED3.A, LS2.C1, PNP.C2, R11.2, R12.1, R19.2, U$2.VCC, U$2.VM
- net ANTENNA: now also R16.1; no longer C26.1
- net GND: now also C21.2, J2.GND@3, J2.GND@5, J2.GNDDTCT, MICROCONTROLLER.38, NPN.E1, NPN.E2, R17.2, R24.2, SUPERCAPACITOR.-, U$1.GND1, U$1.GND2, U$1.GND3, U$3.GND1, U$3.GND2, U$3.GND3; no longer C13.2, C14.2, C15.2, C16.2, C17.2, IMU.GND, IMU.RES, R7.2, U$9.1, U$9.FOOT1, U$9.FOOT2, U$9.FOOT3, U$9.FOOT4
- net JTAG_TCKC: now also J2.SWDCLK/TCK; no longer U$9.14, U$9.15
- net JTAG_TMSC: now also J2.SWDIO/TMS; no longer U$9.16, U$9.17
- net N$15: now also R23.2; no longer GPS.RFIN
- net RESET: now also J2.!RESET; no longer U$9.6, U$9.7
- net RXD: no longer U$9.2, U$9.3
- net SCL: now also SI7021.SCL
- net SDA: now also SI7021.SDA
- net SOLAR_CELLS: now also SCHTOKKY.A; no longer C22.1, L4.2, U$8.SHDN
- net SWO: no longer U$9.8, U$9.9
- net TDI: now also J2.NC/TDI; no longer U$9.10, U$9.11
- net TDO: now also J2.SWO/TDO; no longer U$9.12, U$9.13
- net TXD: no longer U$9.4, U$9.5
- net VDDS: now also C21.1, J2.VCC, PNP.E2, R14.1, SI7021.VDD; no longer GPS.VCC@2, GPS.VCC@58, LED3.A, LS1.C1, LS2.C1, R11.2, R12.1, R19.2, U$2.VCC, U$2.VM, U$9.18, U$9.19
Other:
- note added: "Done: New solar cells Schtokky diode Supercap Humidity sensor ADC changes Remove a light sensor New VCC for GPS (sans vbatt) New VCC for light sensor VBATT for GPS Ground IOID 22 in prototype Transistor arrangement for sensor VCC VCC change for I2C pullups VCC for torque coil driver (?) Unique VCC/GND for IMU and T/H Tuning pads for antennas Change to more convenient transistor control pin"
- note added: "Light Sensor"
- note added: "Temperature and Humidity"
- note added: "To do: Breakout area (?)"
- note removed: "Light Sensors"
- note removed: "Pin Breakouts"
- moved on the sheet: C20, C22, C23, FRONT_PANEL, L4, LS2, R7, R8, REAR_PANEL

Commit message: board layout complete, need to update other files
Parts:
- added LS1: LIGHTSENSORALS, SparkFun-Sensors:LIGHTSENSORALS
- added R26: 10k, SparkFun:RESISTOR0402-RES
- JP1: device SparkFun-Connectors:M14 -> SparkFun:M02PTH
Connections:
- removed net SWO: MICROCONTROLLER.28
- new net ADC2: LS1.E1, MICROCONTROLLER.39, R26.1
- new net CSN: JP2.9, MICROCONTROLLER.21
- new net CTS: JP2.13, MICROCONTROLLER.29
- new net DIO_29: JP2.11, MICROCONTROLLER.42
- new net DIO_30: JP2.10, MICROCONTROLLER.43
- new net MISO: JP2.6, MICROCONTROLLER.14
- new net MOSI: JP2.7, MICROCONTROLLER.15
- new net RTS: JP2.14, MICROCONTROLLER.28
- new net SPICLK: JP2.8, MICROCONTROLLER.16
- net GND: now also JP1.2, R26.2
- net IMUGND: now also JP2.5
- net RXD: now also JP2.1
- net SCL: now also JP2.4
- net SDA: now also JP2.3
- net TXD: now also JP2.2
- net VDDS: now also JP1.1
- net VSENSE: now also JP2.12, LS1.C1
Other:
- note added: "Done: New solar cells Schtokky diode Supercap Humidity sensor ADC changes Remove a light sensor New VCC for GPS (sans vbatt) New VCC for light sensor VBATT for GPS Ground IOID 22 in prototype Transistor arrangement for sensor VCC VCC change for I2C pullups VCC for torque coil driver (?) Unique VCC/GND for IMU and T/H Tuning pads for antennas Change to more convenient transistor control pin Breako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"
- note added: "PROTOTYPE ADC2"
- note added: "To do:"
- note removed: "Done: New solar cells Schtokky diode Supercap Humidity sensor ADC changes Remove a light sensor New VCC for GPS (sans vbatt) New VCC for light sensor VBATT for GPS Ground IOID 22 in prototype Transistor arrangement for sensor VCC VCC change for I2C pullups VCC for torque coil driver (?) Unique VCC/GND for IMU and T/H Tuning pads for antennas Change to more convenient transistor control pin"
- note removed: "To do: Breakout area (?)"
- moved on the sheet: JP2

Commit message: updated all files
Other:
- note added: "Light Sensors"
- note added: "Programming and Pinouts"
- note removed: "Done: New solar cells Schtokky diode Supercap Humidity sensor ADC changes Remove a light sensor New VCC for GPS (sans vbatt) New VCC for light sensor VBATT for GPS Ground IOID 22 in prototype Transistor arrangement for sensor VCC VCC change for I2C pullups VCC for torque coil driver (?) Unique VCC/GND for IMU and T/H Tuning pads for antennas Change to more convenient transistor control pin Breako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"
- note removed: "Light Sensor"
- note removed: "PROTOTYPE ADC2"
- note removed: "To do:"
- moved on the sheet: J2, JP1, JP2

Commit message: RFQ for BSU, changed matching circuit
Parts:
- removed C19: 100pF, SparkFun:CAP0603-CAP
- removed L3: 2.2 nH, SparkFun:INDUCTOR0603
- added L2: 5.6nH, SparkFun:INDUCTOR0603
- added R27: DNP, SparkFun:RESISTOR0603-RES
Connections:
- net ANTENNA: now also R17.2; no longer C19.2
- net GND: now also L2.1, R17.1, R27.2; no longer C19.1, L3.1, R17.2
- net N$15: now also R27.1; no longer L3.2
- net N$26: now also L2.2; no longer R17.1
Other:
- moved on the sheet: R17
Changed lines of the file:
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@@
 <part name="C26" library="SparkFun" deviceset="CAP" device="0402-CAP" value="100 pF"/>
 <part name="GND46" library="SparkFun" deviceset="GND" device=""/>
-<part name="C19" library="SparkFun" deviceset="CAP" device="0603-CAP" value="100pF"/>
-<part name="L3" library="SparkFun" deviceset="INDUCTOR" device="0603" value="2.2 nH"/>
 <part name="GND28" library="SparkFun" deviceset="GND" device=""/>
 <part name="U$5" library="johanson_gps_chip" deviceset="JOHANSON_GPS_CHIP" device=""/>
@@
 <part name="GND36" library="SparkFun" deviceset="GND" device=""/>
 <part name="R16" library="SparkFun" deviceset="RESISTOR" device="0603-RES" value="0"/>
-<part name="R17" library="SparkFun" deviceset="RESISTOR" device="0603-RES" value="DNP"/>
 <part name="R18" library="SparkFun" deviceset="RESISTOR" device="0603-RES" value="DNP"/>
 <part name="R21" library="SparkFun" deviceset="RESISTOR" device="0603-RES" value="0"/>
@@
 <part name="R26" library="SparkFun" deviceset="RESISTOR" device="0402-RES" value="10k"/>
 <part name="LS1" library="SparkFun-Sensors" deviceset="LIGHTSENSOR" device="ALS"/>
+<part name="L2" library="SparkFun" deviceset="INDUCTOR" device="0603" value="5.6nH"/>
+<part name="R17" library="SparkFun" deviceset="RESISTOR" device="0603-RES" value="DNP"/>
+<part name="R27" library="SparkFun" deviceset="RESISTOR" device="0603-RES" value="DNP"/>
 </parts>
 <sheets>
@@
 <attribute name="VALUE" x="37.084" y="109.601" size="1.778" layer="96"/>
 </instance>
-<instance part="GND46" gate="1" x="12.7" y="121.92" rot="R180"/>
-<instance part="C19" gate="G$1" x="12.7" y="111.76" smashed="yes">
-<attribute name="NAME" x="7.874" y="114.2746" size="1.778" layer="95"/>
-<attribute name="VALUE" x="5.08" y="109.982" size="1.778" layer="96"/>
-</instance>
-<instance part="L3" gate="G$1" x="365.76" y="226.06" smashed="yes">
-<attribute name="NAME" x="361.95" y="227.5586" size="1.778" layer="95"/>
-<attribute name="VALUE" x="367.03" y="220.218" size="1.778" layer="96"/>
-</instance>
+<instance part="GND46" gate="1" x="12.7" y="124.46" rot="R180"/>
 <instance part="GND28" gate="1" x="365.76" y="236.22" rot="R180"/>
 <instance part="U$5" gate="G$1" x="365.76" y="200.66" rot="R90"/>
@@
 <attribute name="VALUE" x="14.478" y="104.14" size="1.778" layer="96"/>
 </instance>
-<instance part="R17" gate="G$1" x="22.86" y="111.76" smashed="yes" rot="R90">
-<attribute name="NAME" x="19.5834" y="111.252" size="1.778" layer="95" rot="R90"/>
-<attribute name="VALUE" x="21.844" y="109.728" size="1.778" layer="96" rot="R90"/>
-</instance>
 <instance part="R18" gate="G$1" x="25.4" y="111.76" smashed="yes" rot="R270">
 <attribute name="NAME" x="26.6446" y="115.062" size="1.778" layer="95" rot="R270"/>
@@
 <attribute name="VALUE" x="29.972" y="103.378" size="1.778" layer="96"/>
 </instance>
-<instance part="GND17" gate="1" x="22.86" y="121.92" rot="R180"/>
+<instance part="GND17" gate="1" x="22.86" y="124.46" rot="R180"/>
 <instance part="U$1" gate="G$1" x="40.64" y="119.38"/>
 <instance part="GND18" gate="1" x="60.96" y="116.84"/>
@@
 <attribute name="VALUE" x="40.64" y="142.24" size="1.778" layer="96" rot="R90"/>
 <attribute name="NAME" x="30.48" y="165.1" size="1.778" layer="95"/>
+</instance>
+<instance part="L2" gate="G$1" x="22.86" y="114.3" smashed="yes">
+<attribute name="NAME" x="20.066" y="115.7986" size="1.778" layer="95"/>
+<attribute name="VALUE" x="22.098" y="107.696" size="1.778" layer="96" rot="R90"/>
+</instance>
+<instance part="R17" gate="G$1" x="12.7" y="116.84" smashed="yes" rot="R270">
+<attribute name="NAME" x="13.9446" y="120.142" size="1.778" layer="95" rot="R270"/>
+<attribute name="VALUE" x="16.002" y="121.158" size="1.778" layer="96" rot="R270"/>
+</instance>
+<instance part="R27" gate="G$1" x="365.76" y="223.52" smashed="yes" rot="R90">
+<attribute name="NAME" x="364.2614" y="221.488" size="1.778" layer="95" rot="R90"/>
+<attribute name="VALUE" x="368.808" y="221.742" size="1.778" layer="96" rot="R90"/>
 </instance>
 </instances>
@@
 </segment>
 <segment>
-<pinref part="GND46" gate="1" pin="GND"/>
-<pinref part="C19" gate="G$1" pin="1"/>
-<wire x1="12.7" y1="119.38" x2="12.7" y2="116.84" width="0.1524" layer="91"/>
-</segment>
-<segment>
-<pinref part="L3" gate="G$1" pin="1"/>
-<pinref part="GND28" gate="1" pin="GND"/>
-</segment>
-<segment>
 <pinref part="U$4" gate="G$1" pin="GND"/>
 <pinref part="GND33" gate="1" pin="GND"/>
@@
 <wire x1="279.4" y1="83.82" x2="287.02" y2="83.82" width="0.1524" layer="91"/>
 <pinref part="GND36" gate="1" pin="GND"/>
-</segment>
-<segment>
-<pinref part="R17" gate="G$1" pin="2"/>
-<pinref part="GND17" gate="1" pin="GND"/>
-<wire x1="22.86" y1="119.38" x2="22.86" y2="116.84" width="0.1524" layer="91"/>
 </segment>
 <segment>
@@
 <pinref part="GND31" gate="1" pin="GND"/>
 <pinref part="R26" gate="G$1" pin="2"/>
+</segment>
+<segment>
+<pinref part="GND46" gate="1" pin="GND"/>
+<pinref part="R17" gate="G$1" pin="1"/>
+</segment>
+<segment>
+<pinref part="GND17" gate="1" pin="GND"/>
+<pinref part="L2" gate="G$1" pin="1"/>
+</segment>
+<segment>
+<pinref part="R27" gate="G$1" pin="2"/>
+<pinref part="GND28" gate="1" pin="GND"/>
+<wire x1="365.76" y1="228.6" x2="365.76" y2="233.68" width="0.1524" layer="91"/>
 </segment>
 </net>
@@
 <net name="N$15" class="0">
 <segment>
-<pinref part="L3" gate="G$1" pin="2"/>
 <pinref part="U$5" gate="G$1" pin="SIG"/>
 <wire x1="365.76" y1="213.36" x2="365.76" y2="218.44" width="0.1524" layer="91"/>
 <pinref part="R23" gate="G$1" pin="2"/>
+<pinref part="R27" gate="G$1" pin="1"/>
 <junction x="365.76" y="218.44"/>
 </segment>
@@
 <wire x1="12.7" y1="17.78" x2="40.64" y2="17.78" width="0.1524" layer="91"/>
 <junction x="12.7" y="17.78"/>
-<pinref part="C19" gate="G$1" pin="2"/>
 <wire x1="12.7" y1="63.5" x2="12.7" y2="106.68" width="0.1524" layer="91"/>
 <junction x="12.7" y="63.5"/>
 <pinref part="R16" gate="G$1" pin="1"/>
-<wire x1="12.7" y1="106.68" x2="12.7" y2="109.22" width="0.1524" layer="91"/>
 <junction x="12.7" y="106.68"/>
+<pinref part="R17" gate="G$1" pin="2"/>
+<wire x1="12.7" y1="111.76" x2="12.7" y2="106.68" width="0.1524" layer="91"/>
 </segment>
 </net>
@@
 <segment>
 <pinref part="R16" gate="G$1" pin="2"/>
-<pinref part="R17" gate="G$1" pin="1"/>
 <pinref part="R21" gate="G$1" pin="1"/>
 <wire x1="22.86" y1="106.68" x2="25.4" y2="106.68" width="0.1524" layer="91"/>
-<junction x="22.86" y="106.68"/>
 <pinref part="R18" gate="G$1" pin="2"/>
 <junction x="25.4" y="106.68"/>
-</segment>
-</net>
+<pinref part="L2" gate="G$1" pin="2"/>
+<junction x="22.86" y="106.68"/>
+</segment>
+</net>

Commit message: BSU suggestions
Parts:
- added JP3: (no value), SparkFun:M02PTH
- added R28: 0, SparkFun:RESISTOR0603-RES
Connections:
- new net N$51: R28.2, U$4.VCC
- net SOLAR_CELLS: now also JP3.1
- net SUPERCAP: now also JP3.2, R28.1
- net VDDS: no longer U$4.VCC
Changed lines of the file:
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@@
 <part name="R17" library="SparkFun" deviceset="RESISTOR" device="0603-RES" value="DNP"/>
 <part name="R27" library="SparkFun" deviceset="RESISTOR" device="0603-RES" value="DNP"/>
+<part name="JP3" library="SparkFun" deviceset="M02" device="PTH"/>
+<part name="R28" library="SparkFun" deviceset="RESISTOR" device="0603-RES" value="0"/>
 </parts>
 <sheets>
@@
 <instance part="GND33" gate="1" x="233.68" y="20.32" rot="R90"/>
 <instance part="C20" gate="G$1" x="200.66" y="40.64" smashed="yes" rot="R270">
-<attribute name="NAME" x="203.581" y="39.116" size="1.778" layer="95" rot="R270"/>
+<attribute name="NAME" x="199.644" y="43.561" size="1.778" layer="95"/>
 <attribute name="VALUE" x="204.724" y="41.021" size="1.778" layer="96"/>
 </instance>
@@
 <attribute name="NAME" x="364.2614" y="221.488" size="1.778" layer="95" rot="R90"/>
 <attribute name="VALUE" x="368.808" y="221.742" size="1.778" layer="96" rot="R90"/>
+</instance>
+<instance part="JP3" gate="G$1" x="157.48" y="134.62"/>
+<instance part="R28" gate="G$1" x="200.66" y="30.48" smashed="yes">
+<attribute name="NAME" x="197.358" y="31.7246" size="1.778" layer="95"/>
+<attribute name="VALUE" x="197.104" y="28.448" size="1.778" layer="96"/>
 </instance>
 </instances>
@@
 </segment>
 <segment>
-<pinref part="U$4" gate="G$1" pin="VCC"/>
-<wire x1="205.74" y1="30.48" x2="195.58" y2="30.48" width="0.1524" layer="91"/>
-<label x="195.58" y="30.48" size="1.778" layer="95"/>
-<pinref part="C20" gate="G$1" pin="1"/>
-<wire x1="205.74" y1="40.64" x2="205.74" y2="30.48" width="0.1524" layer="91"/>
-<junction x="205.74" y="30.48"/>
-</segment>
-<segment>
 <pinref part="U$8" gate="G$1" pin="FB"/>
 <wire x1="198.12" y1="66.04" x2="198.12" y2="73.66" width="0.1524" layer="91"/>
@@
 <label x="144.78" y="139.7" size="1.778" layer="95"/>
 </segment>
+<segment>
+<pinref part="C20" gate="G$1" pin="1"/>
+<wire x1="205.74" y1="40.64" x2="215.9" y2="40.64" width="0.1524" layer="91"/>
+<label x="213.36" y="40.64" size="1.778" layer="95"/>
+</segment>
 </net>
 <net name="DCDC_SW" class="0">
@@
 <label x="182.88" y="73.66" size="1.778" layer="95" rot="R270"/>
 <pinref part="SCHTOKKY" gate="G$1" pin="A"/>
+</segment>
+<segment>
+<pinref part="JP3" gate="G$1" pin="1"/>
+<wire x1="165.1" y1="134.62" x2="175.26" y2="134.62" width="0.1524" layer="91"/>
+<label x="167.64" y="134.62" size="1.778" layer="95"/>
 </segment>
 </net>
@@
 <label x="124.46" y="68.58" size="1.778" layer="95"/>
 </segment>
+<segment>
+<pinref part="JP3" gate="G$1" pin="2"/>
+<wire x1="165.1" y1="137.16" x2="175.26" y2="137.16" width="0.1524" layer="91"/>
+<label x="167.64" y="137.16" size="1.778" layer="95"/>
+</segment>
+<segment>
+<pinref part="R28" gate="G$1" pin="1"/>
+<wire x1="195.58" y1="30.48" x2="190.5" y2="30.48" width="0.1524" layer="91"/>
+<wire x1="190.5" y1="30.48" x2="190.5" y2="45.72" width="0.1524" layer="91"/>
+<label x="190.5" y="35.56" size="1.778" layer="95" rot="R90"/>
+</segment>
 </net>
 <net name="VSENSE" class="0">
@@
 </segment>
 </net>
+<net name="N$51" class="0">
+<segment>
+<pinref part="U$4" gate="G$1" pin="VCC"/>
+<pinref part="R28" gate="G$1" pin="2"/>
+</segment>
+</net>
