File: Eagle/Sprite_CC1310_Development.brd (EAGLE design)
At the start: 50 x 50 mm, 59 parts

Commit message: updated JTAG and UART pinouts
Parts:
- removed U$9: HDMID, HDMID:HDMID
- added J1: CORTEX_DEBUG_SMD, SparkFun-Connectors:SAMTECH_FTSH-105-01
- added JP1: (no value), SparkFun:1X02
Connections:
- net GND: now also J1.3, J1.5, J1.9; no longer U$9.1, U$9.FOOT1, U$9.FOOT2, U$9.FOOT3, U$9.FOOT4
- net JTAG_TCKC: now also J1.4; no longer U$9.14, U$9.15
- net JTAG_TMSC: now also J1.2; no longer U$9.16, U$9.17
- net RESET: now also J1.10; no longer U$9.6, U$9.7
- net RXD: now also JP1.1; no longer U$9.2, U$9.3
- net SWO: no longer U$9.8, U$9.9
- net TDI: now also J1.8; no longer U$9.10, U$9.11
- net TDO: now also J1.6; no longer U$9.12, U$9.13
- net TXD: now also JP1.2; no longer U$9.4, U$9.5
- net VDDS: now also J1.1; no longer U$9.18, U$9.19
Routing:
- net RXD: track 46.0 -> 25.4 mm
- net TXD: track 38.2 -> 24.1 mm, vias 2 -> 1
- net VDDS: track 120.0 -> 133.2 mm, vias 13 -> 12
- net SWO: track 12.6 -> 0.00 mm
- net GND: track 181.2 -> 179.0 mm
- net JTAG_TMSC: track 13.4 -> 12.1 mm
- net JTAG_TCKC: track 12.8 -> 11.8 mm
- net TDO: track 12.7 -> 12.1 mm
